Commit message: added color

File: src/robot_arm/urdf/materials.xacro (robot description, xacro)
@@ -1,6 +1,15 @@
 <?xml version="1.0" ?>
 <robot name="robot_arm" xmlns:xacro="http://www.ros.org/wiki/xacro" >
-<material name="silver">
-  <color rgba="0.700 0.700 0.700 1.000"/>
-</material>
+  <!-- Black color -->
+  <material name="black">
+    <color rgba="0.1 0.1 0.1 1.0"/>
+  </material>
+  <!-- Yellow color -->
+  <material name="yellow">
+    <color rgba="1.0 1.0 0.0 1.0"/>
+  </material>
+  <!-- Ash color -->
+  <material name="ash">
+    <color rgba="1.0 0.0 0.0 1.0"/>
+  </material>
 </robot>

File: src/robot_arm/urdf/robot_arm.xacro (robot description, xacro)
@@ -15,5 +15,5 @@
       <mesh filename="file://$(find robot_arm)/meshes/base_link.stl" scale="0.001 0.001 0.001"/>
     </geometry>
-    <material name="silver"/>
+    <material name="black"/>
   </visual>
   <collision>
@@ -35,5 +35,5 @@
       <mesh filename="file://$(find robot_arm)/meshes/shoulder_link_1.stl" scale="0.001 0.001 0.001"/>
     </geometry>
-    <material name="silver"/>
+    <material name="yellow"/>
   </visual>
   <collision>
@@ -55,5 +55,5 @@
       <mesh filename="file://$(find robot_arm)/meshes/elbow_link_1.stl" scale="0.001 0.001 0.001"/>
     </geometry>
-    <material name="silver"/>
+    <material name="ash"/>
   </visual>
   <collision>
